File: boards/trashotron-optical-neuron.sch (EAGLE design)
At the start: 17 parts, among them U1 LM358, U2 LM358, U3 LM358

Commit message: this version of the boards is now all tested out on solderless breadboard
Parts:
- added C1, C2: (no value), rcl:C-EU050-050X075
Connections:
- removed net N$11: D5.C, R6.1, U3G1.+IN
- removed net N$13: D3.C, R4.1, U2G1.+IN
- removed net N$9: D4.C, R5.1, U3G2.+IN
- new net N$4: D3.C, R4.1, U2G1.-IN
- new net N$5: D2.C, R3.1, U2G2.-IN
- new net N$6: D4.C, R5.1, U3G2.-IN
- net GND: now also C1.1, C2.1, U1G1.+IN, U1G2.+IN, U2G1.+IN, U2G2.+IN, U3G1.+IN, U3G2.+IN; no longer U1G1.-IN, U1G2.-IN, U2G1.-IN, U2G2.-IN, U3G1.-IN, U3G2.-IN
- net N$1: now also U1G1.-IN; no longer U1G1.+IN
- net N$7: now also D5.C, R6.1, U3G1.-IN; no longer D2.C, R3.1, U2G2.+IN
- net N$8: now also U1G2.-IN; no longer U1G2.+IN
- net VCC: now also C1.2, C2.2
Other:
- moved on the sheet: D1, D2, D3, D4, D5, D6, R3, R4, R5, R6, R7, R8
