File: boards/trashotron-slimezistor.brd (EAGLE design)
At the start: 50.8 x 25.4 mm, 10 parts, among them U1 LM358

Commit message: this version of the boards is now all tested out on solderless breadboard
Parts:
- added C1: (no value), rcl:C050-050X075
- added R1: (no value), SparkFun-Resistors:AXIAL-0.3
- moved J2 5.08 mm to (48.9, 23.5), turned to 180 degrees
- moved J7 5.08 mm to (48.9, 1.91), turned to 180 degrees
- moved R2 1.90 mm to (12.7, 3.81)
Connections:
- net GND: now also C1.2
- net N$10: now also R1.P$1
- net VCC: now also C1.1, R1.P$2
Routing:
- net N$16: track 13.5 -> 20.1 mm
- net N$12: track 37.0 -> 40.6 mm
- net VCC: track 24.3 -> 27.5 mm
- net N$10: track 14.6 -> 17.3 mm
- net N$5: track 39.9 -> 38.4 mm
- net N$14: track 11.7 -> 12.5 mm
Other:
- board text added: "0.47 uF"
- board text added: "10 kOhm"
- board text added: "github.com/lafelabs/trashotron"
- board text removed: "4.7 kOhm"
